Commit message: test 1

File: urdf/R1Mk3/robots/R1Mk3Gazebo/model.urdf (robot description, URDF)
Before this commit: robot R1Mk3, 182 links, 181 joints
Links:
- link mobile_base_body_link: geometry collision mesh filename=package://R1Mk3/meshes/simmechanics/sim_cer_mobilebase_body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 scale=0.001 0.001 0.001; visual mesh filename=package://R1Mk3/meshes/simmechanics/sim_cer_mobilebase_body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 scale=0.001 0.001 0.001

Commit message: test 4 - base weight

File: urdf/R1Mk3/robots/R1Mk3Gazebo/model.urdf (robot description, URDF)
Before this commit: robot R1Mk3, 182 links, 181 joints
Links:
- link mobile_base_body_link: mass 22.387788717205595 -> 122.387788717205595
